File: hardware/kicad/TORANEKO.Mk3/TORANEKO.Mk3.kicad_pcb (KiCad board)
At the start: 2 copper layers, 54.9 x 64 mm, 93 parts, among them IC1 MP6551GQB-P, IC2 MP6551GQB-P, IC3 NCR321PASX, IC4 NCR321PASX, IC5 AS5047P-ATSM, IC6 STM32F411CEU6TR, IC7 AS5047P-ATSM, IC8 NCR321PASX, IC9 NCR321PASX, J1 Conn_01x02_Pin, J2 Conn_01x02_Pin, J3 Conn_01x02_Male, J4 Conn_01x02_Pin, J5 Conn_01x02_Pin, J6 Conn_02x03_Odd_Even, Q1 IRLML6402, Q5 IRLML6344, SW1 SW_Push, U1 LSM6DSRXTR, U2 LXDC55FAAA-203, U3 Encord, U4 Encord_B, U5 Encord, U6 Encord_B, Y1 CSTNE10M0G52Z000R0

Commit message: Fix capacitor values in TORANEKO.Mk3 schematic/PCB (0.1 -> 0.1u, 10 -> 10u)
- Add missing "u" unit to two 0.1u and two 10u capacitor values
- Sync updated values to the PCB

Co-Authored-By: Claude Opus 5.5 <noreply@anthropic.com>
Changed lines of the file:
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@@
 		(layer "Edge.Cuts")
 	)
-	(gr_line
-		(start 90.9 72.55)
-		(end 90.9 72.550001)
-		(stroke
-			(width 0.2)
-			(type default)
-		)
-		(layer "Edge.Cuts")
-	)
 	(gr_circle
 		(center 121.8 62.3)
@@
 	)
 	(gr_line
-		(start 95.5 72.55)
-		(end 95.5 72.550001)
-		(stroke
-			(width 0.2)
-			(type default)
-		)
-		(layer "Edge.Cuts")
-	)
-	(gr_line
 		(start 124.299998 59.550001)
 		(end 128.899997 59.550001)
@@
 	)
 	(gr_line
-		(start 95.5 72.550001)
-		(end 90.9 72.550001)
+		(start 95.5 72.55)
+		(end 90.9 72.55)
 		(stroke
 			(width 0.2)
@@
 			"1eb49b79-715e-47e2-8335-bc5fb55ff6ee" "209ea889-41fd-4656-a26c-4370938e2779"
 			"3be21da0-84e4-4fc9-af8b-d8b4922ee3fc" "3ebd0218-ae70-4a7a-b71c-5d67d96ee32e"
-			"4082ffeb-8b38-4944-a7a2-3b86d0d451e4" "4089c2f1-dafa-491c-8e58-ed2f086da6a7"
-			"41b550f2-7463-47d6-9373-f283db4b6e37" "42af35a6-3846-4d03-8ec8-d55cb54c5b54"
-			"4534d848-f7ee-4507-be78-5dbc4b2fdc75" "45d5f8bf-0b13-44cb-a301-57b8b8ac0071"
-			"45f9a1d8-3f9a-42ac-b7d3-18af35268afd" "4d64437c-39d3-463c-be97-ebcdfdbf50fd"
+			"4089c2f1-dafa-491c-8e58-ed2f086da6a7" "41b550f2-7463-47d6-9373-f283db4b6e37"
+			"42af35a6-3846-4d03-8ec8-d55cb54c5b54" "4534d848-f7ee-4507-be78-5dbc4b2fdc75"
+			"45d5f8bf-0b13-44cb-a301-57b8b8ac0071" "45f9a1d8-3f9a-42ac-b7d3-18af35268afd"
 			"4f15bf0a-7940-4885-842a-6b64118c0e69" "4f633b82-ea5a-4d1b-8bf0-b22668c45f22"
 			"50d38111-89c0-4aa3-b8ff-9171793dcaeb" "55e01217-1ee2-4fa3-9953-8073a1252a53"

Commit message: Continue TORANEKO.Mk3 PCB routing; update pad geometry
- Adjust existing tracks and add routing (1246 -> 1260 segments)
- Update position/size of 12 pads (likely footprint update from library)

Co-Authored-By: Claude Opus 5.5 <noreply@anthropic.com>
Routing:
- net WallLED-2: track 35.4 -> 36.8 mm
- net Net-(IC7-VDD): track 10.3 -> 11.3 mm
- net Net-(IC7-GND): track 15.0 -> 16.1 mm
- net ENCO-SCK: track 28.3 -> 29.3 mm
- net ENCO-MOSI: track 27.4 -> 28.2 mm
- net FunPWM: track 52.9 -> 53.7 mm
- net ENCO-MISO: track 27.7 -> 28.5 mm

Commit message: Continue TORANEKO.Mk3 PCB routing; refill zone
- Rework and add tracks (1260 -> 1272 segments)
- Refill copper zone

Co-Authored-By: Claude Opus 5.5 <noreply@anthropic.com>
Routing:
- net Net-(IC1-OUT2_1): track 8.96 -> 13.0 mm
- net Net-(IC1-OUT1_1): track 12.1 -> 15.3 mm
- net Net-(IC7-GND): track 16.1 -> 13.4 mm
- net Net-(IC7-VDD): track 11.3 -> 9.63 mm
- net VBAT: track 79.6 -> 80.8 mm
- net Net-(IC5-MOSI): track 5.00 -> 4.38 mm
- net Net-(IC7-MOSI): track 5.15 -> 4.60 mm
