File: hardware/kicad/TORANEKO.Mk3/panel/TORANEKO.Mk3_main_panel.kicad_pcb (KiCad board)
At the start: 2 copper layers, 70 x 78 mm, 92 parts, among them IC1 MP6551GQB-P, IC2 MP6551GQB-P, IC3 NCR321PASX, IC4 NCR321PASX, IC6 STM32F411CEU6TR, IC8 NCR321PASX, IC9 NCR321PASX, J1 Conn_01x02_Pin, J2 Conn_01x02_Pin, J3 Conn_01x02_Male, J4 Conn_01x02_Pin, J5 Conn_01x02_Pin, J6 Conn_02x03_Odd_Even, Q1 IRLML6402, Q5 IRLML6344, SW1 SW_Push, U1 LSM6DSRXTR, U2 LXDC55FAAA-203, U4 Encord_B, U6 Encord_B, Y1 CSTNE10M0G52Z000R0

Commit message: C3/C6 (VBAT): 10uF -> 1uF 25V 0402 and add to PCBA BOM
No 0402 10uF part rated >=16V exists, and VBAT is 2S LiPo (8.4V max);
C2 (100uF) remains as bulk capacitance.

Co-Authored-By: Claude Opus 5.5 <noreply@anthropic.com>
Claude-Session: https://claude.ai/code/session_01Cv6KpZe6NLHWQTjQMUz9Sg
Parts:
- C3, C6: value 10 -> 1u
Changed lines of the file:
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@@
 			)
 		)
-		(property "Value" "10"
+		(property "Value" "1u"
 			(at 0 1.16 0)
 			(layer "F.Fab")
@@
 			)
 		)
-		(property "Value" "10"
+		(property "Value" "1u"
 			(at 0 1.16 0)
 			(layer "F.Fab")

Commit message: Q1/Q5: IRLML6402/6344 -> AO3401A/AO3400A (JLC Basic parts)
Same SOT-23 pinout (1=G, 2=S, 3=D) and +-12V Vgs rating; removes two
Extended parts from the PCBA order.

Co-Authored-By: Claude Opus 5.5 <noreply@anthropic.com>
Claude-Session: https://claude.ai/code/session_01Cv6KpZe6NLHWQTjQMUz9Sg
Parts:
- Q1: value IRLML6402 -> AO3401A
- Q5: value IRLML6344 -> AO3400A
Changed lines of the file:
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@@
 			)
 		)
-		(property "Value" "IRLML6344"
+		(property "Value" "AO3400A"
 			(at 0 2.4 0)
 			(layer "F.Fab")
@@
 			)
 		)
-		(property "Value" "IRLML6402"
+		(property "Value" "AO3401A"
 			(at 0 2.4 0)
 			(layer "F.Fab")

Commit message: C9-C14 (+3.3V): 47uF -> 22uF 0603 (JLC Basic C59461)
Co-Authored-By: Claude Opus 5.5 <noreply@anthropic.com>
Claude-Session: https://claude.ai/code/session_01Cv6KpZe6NLHWQTjQMUz9Sg
Parts:
- C10, C11, C12, C13, C14, C9: value 47u -> 22u
Changed lines of the file:
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@@
 			)
 		)
-		(property "Value" "47u"
+		(property "Value" "22u"
 			(at 0 1.43 0)
 			(layer "F.Fab")
@@
 			)
 		)
-		(property "Value" "47u"
+		(property "Value" "22u"
 			(at 0 1.43 90)
 			(layer "F.Fab")
@@
 			)
 		)
-		(property "Value" "47u"
+		(property "Value" "22u"
 			(at 0 1.43 90)
 			(layer "F.Fab")
@@
 			)
 		)
-		(property "Value" "47u"
+		(property "Value" "22u"
 			(at 0 1.43 90)
 			(layer "F.Fab")
@@
 			)
 		)
-		(property "Value" "47u"
+		(property "Value" "22u"
 			(at 0 1.43 0)
 			(layer "F.Fab")
@@
 			)
 		)
-		(property "Value" "47u"
+		(property "Value" "22u"
 			(at 0 1.43 90)
 			(layer "F.Fab")
